File: ESPREMOTE.sch (EAGLE design)
At the start: 38 parts, among them IC1 ESP12SMT, J1 2.1MM DC Jack, Q1 2N7002, Q2 2N7002, Q3 2N7002, Q4 2N7002

Commit message: Fixed ESP12 pinout for v3.1 release
Connections:
- net GPIO4: no longer R2.2
- net GPIO5: now also R2.2
Other:
- note added: "Output 1: GPIO12 Output 2: GPIO13 Output 3: GPIO14 Output 4: GPIO5"
- note added: "V3.1 (2018-03-28)"
- note removed: "Output 1: GPIO12 Output 2: GPIO13 Output 3: GPIO14 Output 4: GPIO4"
- note removed: "V3.0 (2018-03-09)"
Changed lines of the file:
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@@
 <?xml version="1.0" encoding="utf-8"?>
 <!DOCTYPE eagle SYSTEM "eagle.dtd">
-<eagle version="8.6.0">
+<eagle version="8.7.0">
 <drawing>
 <settings>
@@
 <text x="7.62" y="6.858" size="1.778" layer="94">SKU: ESPREMOTE</text>
 <text x="7.62" y="12.7" size="2.794" layer="94">SuperHouse Automation ESP8266 Remote</text>
-<text x="81.28" y="6.858" size="1.778" layer="94">V3.0 (2018-03-09)</text>
+<text x="81.28" y="6.858" size="1.778" layer="94">V3.1 (2018-03-28)</text>
 <text x="35.306" y="6.858" size="1.778" layer="94">www.superhouse.tv/espremote</text>
 <frame x1="5.08" y1="5.08" x2="109.22" y2="17.78" columns="0" rows="0" layer="94" border-left="no" border-top="no" border-right="no" border-bottom="no"/>
@@
 Output 2: GPIO13
 Output 3: GPIO14
-Output 4: GPIO4</text>
+Output 4: GPIO5</text>
 <text x="38.1" y="48.26" size="1.778" layer="97">Output 1</text>
 <text x="38.1" y="45.72" size="1.778" layer="97">Output 2</text>
@@
 <segment>
 <pinref part="IC1" gate="G$1" pin="GPIO5"/>
-<wire x1="93.98" y1="53.34" x2="121.92" y2="53.34" width="0.1524" layer="91"/>
-<label x="111.76" y="53.34" size="1.778" layer="95"/>
-</segment>
-</net>
-<net name="GPIO4" class="0">
-<segment>
-<pinref part="IC1" gate="G$1" pin="GPIO4"/>
-<wire x1="93.98" y1="55.88" x2="124.46" y2="55.88" width="0.1524" layer="91"/>
+<wire x1="93.98" y1="55.88" x2="121.92" y2="55.88" width="0.1524" layer="91"/>
 <label x="111.76" y="55.88" size="1.778" layer="95"/>
 </segment>
@@
 </segment>
 </net>
+<net name="GPIO4" class="0">
+<segment>
+<pinref part="IC1" gate="G$1" pin="GPIO4"/>
+<wire x1="93.98" y1="53.34" x2="121.92" y2="53.34" width="0.1524" layer="91"/>
+<label x="111.76" y="53.34" size="1.778" layer="95"/>
+</segment>
+</net>
